File: BreakoutBoards/LED_RGB/LED_RGB.kicad_pcb (KiCad board)
At the start: 2 copper layers, 11.3 x 12.8 mm, 7 parts, among them J1 Conn_01x04_Pin

Commit message: tweaked silkscreen positions
Other:
- board text added: "ChargeForge LED_RGB Mk 0.1"
- board text removed: "ChargeForge LED_RGB Mk0.1"
Changed lines of the file:
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@@
 		)
 		(pad_to_mask_clearance 0)
-		(solder_mask_min_width 0.12)
 		(allow_soldermask_bridges_in_footprints no)
 		(tenting front back)
@@
 		)
 	)
-	(gr_text "ChargeForge\nLED_RGB Mk0.1"
-		(at 97.78541 94.488704 0)
+	(gr_text "ChargeForge\nLED_RGB Mk 0.1"
+		(at 97.85 94.476 0)
 		(layer "B.SilkS")
 		(effects
@@
 	)
 	(gr_text "Copyright © 2026 clectric.diy\nLicensed under CERN-OHL-W v2"
-		(at 97.88541 96.188704 0)
+		(at 97.88 95.91 0)
 		(layer "B.SilkS")
 		(effects
