File: BreakoutBoards/Potentiometer_RGB-3.3V/KiCad/Potentiometer_RGB-3.3V/Potentiometer_RGB-3.3V.kicad_sch (KiCad schematic)
At the start: 2 parts, among them J1 Conn_01x06_Pin

Commit message: updated to Mk1 and sent for manufacturing
Parts:
- added R1, R3: 27R, clectric-diy:R0603, symbol Device:R
- added R2: 75R, clectric-diy:R0603, symbol Device:R
- added U2: A-SP1943B1GHR6C-C01-2T, clectric-diy:LED-SMD_4P-L1.6-W1.5-BL_A-SP1943B1GHR6C-C01-2T, symbol clectric-diy:A-SP1943B1GHR6C-C01-2T
- J1: footprint clectric-diy:HDR-TH_6P-P2.54-V-M-1 -> Connector_PinHeader_2.54mm:PinHeader_1x06_P2.54mm_Vertical
Connections:
- net LED_BLUE: now also R3.1, R3.2, U2.4
- net LED_GREEN: now also R1.1, R1.2, U2.1
- net LED_RED: now also R2.1, R2.2, U2.2
- net VCC+CW renamed 3.3V+CW
- net 3.3V+CW: now also U2.3
Other:
- title: Charge Potentiometer_RGB -> Charge Potentiometer & 3.3V RGB LED
- moved on the sheet: J1, R4
